File: Electrical/Schematics/KiCad_Project/01_Ana_Guc_24VDC.kicad_sch (KiCad schematic)
At the start: 0 parts

Commit message: feat: update electrical schematics to rev 4.0, add technical manuals, and include project documentation and validation reports.
Parts:
- added X1: AC_Giris_3F400V, TerminalBlock:TerminalBlock_Phoenix_MKDSN-2,5-5_1x05, symbol Connector_Generic:Conn_01x05
- added X2: 24V_Dagitim, TerminalBlock:TerminalBlock_Phoenix_MKDSN-2,5-5_1x08, symbol Connector_Generic:Conn_01x08
Connections:
- new net +24V_NC300: X2.?
Other:
- note added: "24VDC POWER SUPPLY"
- note added: "3-Faz 400VAC Giris -> Kontaktor -> 24VDC PSU -> X2 Dagitim"
- note added: "AC GIRIS (3F 400VAC)"
- note added: "AC Guc: 6mm² (L1/L2/L3), 4mm² (N), 10mm² (PE)"
- note added: "DC Guc: 2.5mm² (+24V), 2.5mm² (0V)"
- note added: "F1 - SIGORTA (3A)"
- note added: "F2: 3A - NC300"
- note added: "F3: 5A - R1-EC I/O"
- note added: "F4: 1A - HMI"
- note added: "F5: 3A - SENSORS"
- note added: "F6: 2A - SAFETY"
- note added: "Input: 3F 400VAC | Output: 24VDC / 20A"
- note added: "K1 - KONTAKTOR (24VDC coil)"
- note added: "Kablo Kesitleri:"
- note added: "L1"
- note added: "L2"
- note added: "L3"
- note added: "N"
- note added: "PE"
- note added: "PS1: 24VDC / 20A (Siemens SITOP PSU8200)"
- note added: "Q1 - Ana SALTER (32A 3P)"
- note added: "SIGORTA DAGITIMI (24VDC)"
- note added: "Sinyal: 1.0mm² (sensör, kontrol)"
- note added: "X2 DAGITIM TERMINALI"
- note removed: "+24V GLOBAL BUS"
- note removed: "0V GLOBAL BUS"
- note removed: "Bu sayfa guc omurgasini ERC temiz olacak sekilde kurar: +24V, 0V ve PE referanslari. X2 dagitim terminali ve alanlar not olarak korunur."
- note removed: "PE / SHIELD BAR"
- note removed: "PE baglantisi terminal/bara seviyesinde uygulanacak."
- note removed: "PS1 24VDC POWER SUPPLY"
- note removed: "PS1.1 -> +24V bus PS1.2 -> 0V bus XPE1 -> PE / shield barasi"
- note removed: "X2 DAGITIM TERMINAL PLAN"
- note removed: "X2.1 +24V_NC300 X2.2 +24V_R1EC X2.3 +24V_SENS X2.4 +24V_SAFETY X2.5 +24V_HMI X2.6 0V_COMMON X2.7 0V_SENS X2.8 PE_SHIELD"
- company: CNCRevizyon -> CNCRevizyon - GFB60/30RE-S
