File: Electrical/Schematics/KiCad_Project/02_Emniyet_STO.kicad_sch (KiCad schematic)
At the start: 3 parts, among them K1 Pilz_PNOZ_X2_8P, X10 Safety_Inputs, X11 STO_Outputs

Commit message: feat: update electrical schematics to rev 4.0, add technical manuals, and include project documentation and validation reports.
Parts:
- removed K1: Pilz_PNOZ_X2_8P, symbol Connector_Generic:Conn_01x08
- removed X11: STO_Outputs, symbol Connector_Generic:Conn_01x08
- added X11: STO_Outputs, TerminalBlock:TerminalBlock_Phoenix_MKDSN-2,5-5_1x12, symbol Connector_Generic:Conn_01x12
- X10: footprint (none) -> TerminalBlock:TerminalBlock_Phoenix_MKDSN-2,5-5_1x06
Other:
- note added: "- E-STOP butonu 2-kanalli, NC kontaklar kullanilir"
- note added: "- Feedback devresi: Tum STO kontaklari seri, 41-42'ye bagli"
- note added: "- Guvenlik kapisi NC kontak, seri bagli"
- note added: "- Reset butonu NO, manual reset"
- note added: "- STO kablosu: Shielded twisted pair"
- note added: "- STO: Safe Torque Off, 24VDC, 10mA per channel"
- note added: "13-14: Safety Output 1 (N/O) -> STO_A (tum eksenler)"
- note added: "23-24: Safety Output 2 (N/O) -> STO_B (tum eksenler)"
- note added: "33-34: Safety Output 3 (N/O) -> SERVO_ENABLE"
- note added: "41-42: Auxiliary Output (N/C) -> Feedback"
- note added: "A1: +24VDC | A2: 0V"
- note added: "CH1 (Yesil): Channel 1 active"
- note added: "CH2 (Yesil): Channel 2 active"
- note added: "E-STOP GIRISLERI (2-KANAL)"
- note added: "ERR (Kirmizi): Fault detected"
- note added: "GUVENLIK NOTLARI:"
- note added: "K1 - Safety Relay"
- note added: "LED GOSTERGELERI"
- note added: "OUT (Yesil): Safety outputs ON"
- note added: "PILZ PNOZ X2.8P"
- note added: "PWR (Yesil): Power ON"
- note added: "Pilz PNOZ X2.8P Safety Relay - 2-Kanal E-STOP - STO Dagitim"
- note added: "S11: CH1 Input"
- note added: "S12: CH2 Input"
- note added: "S34: Test Pulse"
- note added: "S52: Reset Input"
- note added: "SAFETY CIKIS KONTAKLARI"
- note added: "STO CIKISLARI (5 EKSEN)"
- note added: "X10.1: E-STOP CH1 (NC)"
- note added: "X10.2: E-STOP CH2 (NC)"
- note added: "X10.3: DOOR SAFE (NC)"
- note added: "X10.4: RESET BTN (NO)"
- note added: "X10.5: +24V_SAFETY"
- note added: "X10.6: 0V_SAFETY"
- note added: "X11.1-2: STO X (STO_A_X, STO_B_X)"
- note added: "X11.11: SAFE_FB (Feedback)"
- note added: "X11.12: SERVO_ENABLE_CHAIN"
- note added: "X11.3-4: STO Y (STO_A_Y, STO_B_Y)"
- note added: "X11.5-6: STO Z (STO_A_Z, STO_B_Z)"
- note added: "X11.7-8: STO ALT (STO_A_ALT, STO_B_ALT)"
- note added: "X11.9-10: STO CNC (STO_A_CNC, STO_B_CNC)"
- note removed: "X10 girisleri K1 safety bloguna, K1 de X11 STO cikislarina baglandi."
- note removed: "X10.1 E-STOP CH1 X10.2 E-STOP CH2 X10.3 DOOR SAFE X10.4 RESET X10.5 +24V SAFETY X10.6 0V SAFETY"
- note removed: "X11.1 STO_A_X X11.2 STO_B_X X11.3 STO_A_Y X11.4 STO_B_Y X11.5 STO_A_Z X11.6 STO_B_Z X11.7 SAFE_FB X11.8 SERVO_ENABLE_CHAIN"
- company: CNCRevizyon -> CNCRevizyon - GFB60/30RE-S
