File: Electrical/Schematics/KiCad_Project/03_NC300_EtherCAT.kicad_sch (KiCad schematic)
At the start: 0 parts

Commit message: feat: update electrical schematics to rev 4.0, add technical manuals, and include project documentation and validation reports.
Parts:
- added CN1: EtherCAT_IN, Connector_RJ:RJ45_Amphenol_54601-x0x, symbol Connector:RJ45
- added CN3: HMI_Ethernet, Connector_RJ:RJ45_Amphenol_54601-x0x, symbol Connector:RJ45
- added CN5: NC300_IO_50pin, Connector_Dsub:DSUB-50_Male, symbol Connector_Generic:Conn_01x16
- added PWR_NC300: 24VDC_2A, symbol Connector_Generic:Conn_01x02
Other:
- note added: "+24V (2A max) -> CN5 Pin 1"
- note added: "0V (GND) -> CN5 Pin 18"
- note added: "CN1: EtherCAT IN (RJ45) -> X Ekseni CN3"
- note added: "CN2: EtherCAT OUT (RJ45) <- CNC Ekseni CN6 (loop-back)"
- note added: "CN3: HMI Ethernet (RJ45, 10/100 Mbps)"
- note added: "Cycle Time: 1ms (5 servo + I/O)"
- note added: "DI_0 (Pin 2): SERVO_READY"
- note added: "DI_1 (Pin 3): CYCLE_START"
- note added: "DI_2 (Pin 4): CYCLE_STOP"
- note added: "DI_3 (Pin 5): HOME_CMD"
- note added: "DI_4 (Pin 6): E-STOP_FB"
- note added: "DO_0 (Pin 10): SYSTEM_READY"
- note added: "DO_1 (Pin 11): CYCLE_ACTIVE"
- note added: "DO_2 (Pin 12): ALARM_LIGHT"
- note added: "Delta NC300 CNC Controller - Ana Kontrolor"
- note added: "ETHERCAT DAISY-CHAIN TOPOLOJISI"
- note added: "ETHERCAT MASTER PORTLARI"
- note added: "FG (Frame Ground) < 100Ω to earth"
- note added: "GROUNDDING"
- note added: "HMI ETHERNET BAGLANTISI"
- note added: "HMI: Delta DOP-110CS"
- note added: "Kablo: CAT6 shielded, endustriyel"
- note added: "Kablo: Min 2mm², direkt topraklama"
- note added: "NC300 GUC BAGLANTISI"
- note added: "NC300 YEREL I/O (CN5 - 50pin D-Sub)"
- note added: "Node 0: NC300 (Master)"
- note added: "Node 1: X Ekseni (ASD-A3-4523-E, 4.5kW)"
- note added: "Node 2: Y Ekseni (ASD-A3-2023-E, 2.0kW)"
- note added: "Node 3: ALT Ekseni (ASD-A3-2023-E, 2.0kW)"
- note added: "Node 4: Z Ekseni (ASD-A3-1023-E, 1.0kW, Frenli)"
- note added: "Node 5: CNC Ekseni (ASD-A3-1523-E, 1.5kW)"
- note added: "Node 6: R1-EC Coupler (I/O Genisleme)"
- note added: "Protokol: Delta TCP veya Modbus TCP"
- note added: "Sigorta: F2 (3A slow-blow)"
- note removed: "Plan: - Delta NC300 kontrolor - EtherCAT master portlari - HMI Ethernet baglantisi - X30/X31 network ve alarm/enable ozetleri"
- note removed: "Slave sirasi: X -> Y -> ALT -> Z -> CNC -> R1-EC"
- company: CNCRevizyon -> CNCRevizyon - GFB60/30RE-S
