File: Electrical/Schematics/KiCad_Project/04_Servo_Suruculer.kicad_sch (KiCad schematic)
At the start: 0 parts

Commit message: feat: update electrical schematics to rev 4.0, add technical manuals, and include project documentation and validation reports.
Other:
- note added: "04 - Servo Suruculer (5 Eksen)"
- note added: "CN1 I/O PINOUT (50-pin D-Sub)"
- note added: "CN1 Pin 40: BRK (Fren kontrol)"
- note added: "CN1: STO1/STO2 (Pin 29/30), S-ON (Pin 6)"
- note added: "CN1: STO1/STO2, S-ON"
- note added: "CN2: Encoder (6-pin, 24-bit absolute)"
- note added: "CN3/CN6: EtherCAT IN/OUT (RJ45)"
- note added: "Delta ASDA-A3-E EtherCAT Servo Suruculer"
- note added: "EKSEN 1: X (4.5kW YUKSEK ATalet)"
- note added: "EKSEN 2: Y (2.0kW ORTA ATalet)"
- note added: "EKSEN 3: ALT (2.0kW ORTA ATalet)"
- note added: "EKSEN 4: Z (1.0kW FRENLI)"
- note added: "EKSEN 5: CNC/RODAJ (1.5kW)"
- note added: "Fren: 24VDC, 0.35A, 8.4W (DO_5 kontrol)"
- note added: "Kablo: Shielded twisted pair"
- note added: "Kaynak: Pilz PNOZ X2.8P (13-14, 23-24)"
- note added: "Motor: ECMA-C11010FS (1.0kW, FRENLI)"
- note added: "Motor: ECMA-E11315 (1.5kW, IP67)"
- note added: "Motor: ECMA-E11320 (2.0kW, 24-bit encoder)"
- note added: "Motor: ECMA-L11845 (4.5kW, 24-bit encoder)"
- note added: "P1: R/L1, S/L2 (1F 230VAC, 10A)"
- note added: "P1: R/S/T (3F 400VAC, 16A)"
- note added: "P1: R/S/T (3F 400VAC, 25A)"
- note added: "P2: U/V/W -> Motor (1.5mm² shielded)"
- note added: "P2: U/V/W -> Motor (2.5mm² shielded)"
- note added: "P2: U/V/W -> Motor (4mm² shielded)"
- note added: "Pin 29-30: STO1/STO2"
- note added: "Pin 36-40: DO_1-DO_5 (Alarm, ZSPD, POS, WARN, BRK)"
- note added: "Pin 43: STO_COM (0V)"
- note added: "Pin 44: COM+ (24V return)"
- note added: "Pin 6: S-ON (Servo ON, aktif low)"
- note added: "Pin 9: +24V (Kontrol gucu)"
- note added: "Rejeneratif: 120Ω / 50W (dahili)"
- note added: "Rejeneratif: 60Ω / 100W (dahili)"
- note added: "Rejeneratif: 60Ω / 50W (dahili)"
- note added: "Rejeneratif: 80Ω / 50W (dahili)"
- note added: "STO BAGLANTILARI (Tum Eksenler)"
- note added: "STO1 (CN1 Pin 29): 24VDC, 10mA"
- note added: "STO2 (CN1 Pin 30): 24VDC, 10mA"
- note added: "STO_COM (CN1 Pin 43): 0V"
- note added: "Surucu: ASD-A3-1023-E (1F 230VAC)"
- note added: "Surucu: ASD-A3-1523-E (1F 230VAC)"
- note added: "Surucu: ASD-A3-2023-E (3F 400VAC)"
- note added: "Surucu: ASD-A3-4523-E (3F 400VAC)"
- note removed: "04 - Servo Suruculer"
- note removed: "Plan: - Her eksen icin guc ve motor baglantisi - EtherCAT IN/OUT - STO ST1/ST2 - Z ekseni fren baglantisi"
- note removed: "Sürücüler: X ASD-A3-4523-E, Y ASD-A3-2023-E, ALT ASD-A3-2023-E, Z ASD-A3-1023-E, CNC ASD-A3-1523-E"
- company: CNCRevizyon -> CNCRevizyon - GFB60/30RE-S
- title: 04 Servo Suruculer -> 04 Servo Suruculer - 5 Eksen Detayli
