File: Electrical/Schematics/KiCad_Project/05_R1EC_IO.kicad_sch (KiCad schematic)
At the start: 0 parts

Commit message: feat: update electrical schematics to rev 4.0, add technical manuals, and include project documentation and validation reports.
Other:
- note added: "%IX0.0: X_HOME"
- note added: "%IX0.1: X_LIMIT_P"
- note added: "%IX0.2: X_LIMIT_N"
- note added: "%IX0.3-5: Y_HOME, Y_LIMIT_P, Y_LIMIT_N"
- note added: "%IX2.0-2: Z_HOME, Z_LIMIT_P, Z_LIMIT_N"
- note added: "%IX2.6: GLASS_DETECT"
- note added: "%IX2.7: VACUUM_FB"
- note added: "%IX2.8: DOOR_SAFE"
- note added: "%QX0.0: SERVO_ENABLE"
- note added: "%QX0.1: VACUUM_PUMP"
- note added: "%QX0.4: WARNING_LIGHT"
- note added: "%QX0.5: BUZZER"
- note added: "Adres: %IX0.0 - %IX1.15"
- note added: "Adres: %IX2.0 - %IX3.15"
- note added: "Adres: %QX0.0 - %QX1.15"
- note added: "Block 1: %IX0.0-%IX0.15 (X/Y HOME, LIMIT)"
- note added: "Block 1: %IX2.0-%IX2.15 (Cam, Vakum, Kapi)"
- note added: "Block 1: %QX0.0-%QX0.15 (Aktuatorler)"
- note added: "Block 2: %IX1.0-%IX1.15 (Z/ALT HOME, LIMIT)"
- note added: "Block 2: %IX3.0-%IX3.15 (Rezerve)"
- note added: "Block 2: %QX1.0-%QX1.15 (Rezerve)"
- note added: "COM: 0V (ortak)"
- note added: "Coil: 24VDC"
- note added: "Cycle Time: 1ms minimum"
- note added: "DI TERMINAL BAGLANTISI (Her 16-li grup)"
- note added: "DO TERMINAL BAGLANTISI (Her 16-li grup)"
- note added: "Delta R1-EC EtherCAT Remote I/O Sistemi"
- note added: "EtherCAT IN: CN3 (RJ45) <- CNC Ekseni CN6"
- note added: "EtherCAT OUT: CN6 (RJ45) -> NC300 CN2 (loop)"
- note added: "Filtre: 1ms hardware"
- note added: "Giris: 24VDC (11-30V), 5-10mA"
- note added: "Guc: 24VDC, 150mA (coupler kendisi)"
- note added: "I/O ADRESLEME OZETI"
- note added: "I/O Besleme: V_IO (harici 24VDC)"
- note added: "Izolasyon: Opto-izole (500V)"
- note added: "MODUL #1: R1-EC0902D (32-CH DI)"
- note added: "MODUL #2: R1-EC0902D (32-CH DI)"
- note added: "MODUL #3: R1-EC0902O (32-CH DO RELAY)"
- note added: "Model: R1-EC01 (EtherCAT Coupler)"
- note added: "R1-EC01 BUS COUPLER"
- note added: "Röle: SPST, 2A, 250VAC/30VDC"
- note added: "Sensor: PNP NO (Leuze IS 218)"
- note added: "Terminal 1-16: DI_0 - DI_15"
- note added: "Terminal 1-16: DO_0 NO/COM - DO_7 NO/COM"
- note added: "Toplam Akim: 8A per module"
- note added: "Valf: +24V -> Valf(+) -> Valf(-) -> DO_X NO -> DO_X COM -> 0V"
- note removed: "Plan: - R1-EC bus coupler - DI: R1-EC0902D x3 - DO: R1-EC0902O x3 - EtherCAT node konumu ve kanal gruplari"
- company: CNCRevizyon -> CNCRevizyon - GFB60/30RE-S
