File: Electrical/Schematics/KiCad_Project/06_Dijital_Girisler.kicad_sch (KiCad schematic)
At the start: 0 parts

Commit message: feat: update electrical schematics to rev 4.0, add technical manuals, and include project documentation and validation reports.
Other:
- note added: "+24V_SENS ──► Sensor Pin 1 (Kahverengi)"
- note added: "06 - Dijital Girisler ve Sensorler"
- note added: "Akım Tuketimi: 20mA (max)"
- note added: "Algılama Mesafesi: 8mm (nominal), 10mm (maks)"
- note added: "BAGLANTI SEMASI (PNP Sensor)"
- note added: "Besleme: 10-30V DC (24VDC nominal)"
- note added: "Boyut: M18 x 1 x 75 mm"
- note added: "Cıkıs Tipi: PNP NO/NC (secilebilir)"
- note added: "Dis Cap: 6.0mm"
- note added: "E-Stop: NC (Guvenlik)"
- note added: "Glass Detect: NO (Cam var/yok)"
- note added: "Home Switch: NO (Referans kenar)"
- note added: "Iletken: 4 x 0.34mm²"
- note added: "KABLO OZELLIKLERI"
- note added: "Konum: X=0mm (home), X=5950mm (+limit), X=-50mm (-limit)"
- note added: "Konum: Y=0mm (home), Y=2950mm (+limit), Y=-50mm (-limit)"
- note added: "Konum: Z=0mm (home), Z=+100mm (+limit)"
- note added: "Koruma Sinifi: IP67, IP68, IP69K"
- note added: "Koruma: IP67, Yaga Dayanikli"
- note added: "Leuze IS 218 Serisi Induktif Sensorler - M12 4-pin"
- note added: "Limit Switch: NC (Guvenlik)"
- note added: "M12 4-PIN KONEKTOR PINOUT"
- note added: "Model: Leuze IS 218 MM / IS 218 AM"
- note added: "NO/NC SECIMI"
- note added: "Pin 1 (Kahverengi): +24V DC"
- note added: "Pin 2 (Beyaz): Output PNP (Sinyal)"
- note added: "Pin 3 (Mavi): 0V DC"
- note added: "Pin 4 (Siyah): NO/NC Select"
- note added: "SENSOR TEKNIK OZELLIKLERI"
- note added: "Sensor Pin 2 (Beyaz) ──► DI_X (R1-EC0902D)"
- note added: "Sensor Pin 3 (Mavi) ──► 0V_SENS"
- note added: "Sensor Pin 4 (Siyah) ──► +24V (NC secimi icin)"
- note added: "Sicaklik: -40°C ... +90°C"
- note added: "Tip: Shielded Sensor Cable"
- note added: "X EKSENI SENSORLERI"
- note added: "X_HOME: %IX0.0 (M12 -> R1-EC0902D DI_0)"
- note added: "X_LIMIT_N: %IX0.2 (M12 -> R1-EC0902D DI_2)"
- note added: "X_LIMIT_P: %IX0.1 (M12 -> R1-EC0902D DI_1)"
- note added: "Y EKSENI SENSORLERI"
- note added: "Y_HOME: %IX0.3 (M12 -> R1-EC0902D DI_3)"
- note added: "Y_LIMIT_N: %IX0.5 (M12 -> R1-EC0902D DI_5)"
- note added: "Y_LIMIT_P: %IX0.4 (M12 -> R1-EC0902D DI_4)"
- note added: "Z EKSENI SENSORLERI"
- note added: "Z_HOME: %IX2.0 (M12 -> R1-EC0902D #2 DI_0)"
- note added: "Z_LIMIT_N: %IX2.2 (M12 -> R1-EC0902D #2 DI_2)"
- note added: "Z_LIMIT_P: %IX2.1 (M12 -> R1-EC0902D #2 DI_1)"
- note removed: "06 - Dijital Girisler ve Sensörler"
- note removed: "Kaynak harita: IX0.0..IX0.15"
- note removed: "Plan: - X/Y/Z/ALT limit ve home sensörleri - E-STOP1, E-STOP2, DOOR, VACUUM - M12 4-pin saha konnektor mantigi - X20 terminal referansi"
- company: CNCRevizyon -> CNCRevizyon - GFB60/30RE-S
- title: 06 Dijital Girisler ve Sensörler -> 06 Dijital Girisler ve Sensorler
