File: Electrical/Schematics/KiCad_Project/07_Dijital_Cikislar.kicad_sch (KiCad schematic)
At the start: 0 parts

Commit message: feat: update electrical schematics to rev 4.0, add technical manuals, and include project documentation and validation reports.
Other:
- note added: "%QX0.0: SERVO_ENABLE (Tum servo enable)"
- note added: "%QX0.1: VACUUM_PUMP (Vakum pompasi)"
- note added: "%QX0.2: CUTTING_OIL (Kesim yagi)"
- note added: "%QX0.3: BLADE_SPIN (Testere dönüsü)"
- note added: "%QX0.4: WARNING_LIGHT (Uyari lambasi)"
- note added: "%QX0.5: BUZZER (Alarm buzzer)"
- note added: "%QX0.6: BREAKER_ENABLE (Salter kontrol)"
- note added: "%QX0.7: CLAMP_PRESS (Cam sikistirma)"
- note added: "+24V ──► Buzzer (+)"
- note added: "+24V ──► Kontaktör A1"
- note added: "+24V ──► Lamba (+)"
- note added: "+24V ──► Valf (+)"
- note added: "BUZZER BAGLANTISI"
- note added: "Buzzer (-) ──► DO_5 NO contact"
- note added: "Buzzer: 24VDC, 85dB"
- note added: "CIKIS ADRESLERI (R1-EC0902O)"
- note added: "Coil Voltaj: 24VDC"
- note added: "DO_0 COM ──► 0V"
- note added: "DO_4 COM ──► 0V"
- note added: "DO_5 COM ──► 0V"
- note added: "DO_X COM ──► 0V"
- note added: "F10: 3A - Valfler (toplam)"
- note added: "F7: 5A - Vakum pompa"
- note added: "F8: 2A - Uyari lambasi"
- note added: "F9: 1A - Buzzer"
- note added: "Flyback diyot: 1N4007 (korumа)"
- note added: "Kontaktör A2 ──► DO_0 NO contact"
- note added: "Kontaktör bobin: 24VDC"
- note added: "Lamba (-) ──► DO_4 NO contact"
- note added: "Lamba: 24VDC, 21W (LED önerilir)"
- note added: "Maks Akim: 2A per channel"
- note added: "Maks Voltaj: 250VAC / 30VDC"
- note added: "RÖLE SPEKSIKASYONLARI"
- note added: "Röle Cikislari - Aktuator Kontrol"
- note added: "SIGURTA DAGITIMI (Cikislar)"
- note added: "Tepki Süresi: < 10ms"
- note added: "Tip: SPST relay (NO contact)"
- note added: "Toplam Akim: 8A per module"
- note added: "UYARI LAMBASI BAGLANTISI"
- note added: "VAKUM POMPA BAGLANTISI"
- note added: "VALF BAGLANTISI (Örnek)"
- note added: "Valf (-) ──► DO_X NO contact"
- note added: "Ömür: 100,000 cycles (min)"
- note removed: "On tanimli cikislar: %QX0.0 SERVO_ENABLE, %QX0.1 VACUUM_PUMP, %QX0.4 WARNING_LIGHT, %QX0.5 BUZZER, %QX0.7 BREAKER_ENABLE"
- company: CNCRevizyon -> CNCRevizyon - GFB60/30RE-S
